File: kicad_board/zigbeebox.kicad_pcb (KiCad board)
At the start: 2 copper layers, 79.7 x 47.1 mm, 31 parts, among them J1 Debug, J2 JLINK-JTAG, SW1 RESET, U1 CC2538+CC2592 MODULE

Commit message: Minor trace width adjustments
Routing:
- net Net-(F1-Pad2): track 58.6 -> 38.5 mm
- net Net-(C1-Pad1): track 9.73 -> 3.86 mm
- net Net-(C5-Pad1): track 51.5 -> 48.5 mm
- net Net-(C2-Pad1): track 90.7 -> 93.4 mm
- net Net-(LED3-Pad1): track 51.4 -> 53.9 mm
- net Net-(R3-Pad2): track 47.1 -> 44.7 mm
- net Net-(C4-Pad1): track 70.1 -> 68.1 mm
- net GND: track 32.8 -> 34.4 mm, vias 5 -> 4
- net Net-(J2-Pad15): track 114.7 -> 115.6 mm
- added copper zone on F.Cu, net Net-(C1-Pad1)
- added copper zone on F.Cu, net Net-(F1-Pad2)
